File: hardware/v1.0_esp32_sensor/Nira_Micro-Plastic_Detection_Sensor/Nira_Micro-Plastic_Detection_Sensor.kicad_sch (KiCad schematic)
At the start: 3 parts, among them U2 DEVKIT_V1_ESP32-WROOM-32

Commit message: schematics pdf added
Parts:
- added D1: LED, symbol Device:LED
- added V1: 3.3V, symbol Simulation_SPICE:VDC
- U1: value ~ -> PC_FDC1004
- U2: Availability Not in stock -> (none); Check_prices https://www.snapeda.com/parts/DEVKIT%20V1%20ESP32-WROOM-32/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 -> (none); MANUFACTURER Espressif Systems -> (none); MF Espressif Systems -> (none); MP DEVKIT V1 ESP32-WROOM-32 -> (none); PARTREV N/A -> (none); Package Package -> (none); Price None -> (none); STANDARD Manufacturer Recommendations -> (none); SnapEDA_Link https://www.snapeda.com/parts/DEVKIT%20V1%20ESP32-WROOM-32/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 -> (none)
Connections:
- net GND: now also D1.1 (K), V1.2
- net LED: now also D1.2 (A)
- net VCC: now also U2.1 (3V3), V1.1
- no-connect marks 32 -> 37
Other:
- company:                 FOSS UNITED -> FOSS UNITED
- title:                 NIRA v1.0 - Micro-plastic Sensor -> NIRA v1.0 - Micro-plastic Sensor
