File: hardware/v1.5_esp32_sensor/Nira_Micro-Plastic_Detection_Sensor/Nira_Micro-Plastic_Detection_Sensor.kicad_sch (KiCad schematic)
At the start: 7 parts, among them M1 Motor_DC, U1 ESP32-DEVKIT-V1

Commit message: docs: standardize versions to v1.5 everywhere and generate Wiki structure
Other:
- title: NIRA v1.0 - Micro-plastic Sensor -> NIRA v1.5 - Micro-plastic Sensor
Changed lines of the file:
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@@
   (paper "A4")
   (title_block
-    (title "NIRA v1.0 - Micro-plastic Sensor")
+    (title "NIRA v1.5 - Micro-plastic Sensor")
     (date "2026-03-23")
-    (rev "v1.0")
+    (rev "v1.5")
     (company "FOSS UNITED")
     (comment 1 "CC-BY-SA 4.0 International")
